Commit message: fix(amr_description): fix gazebo.xacro friction refs, merge duplicate blocks, remove deprecated transmissions
- Merge duplicate <gazebo reference="base_link"> blocks into one
- Fix wheel friction: reference links (wheel_left_link) not joints
- Remove deprecated <transmission> tags (not needed for gz_ros2_control)
- Add conditional joint_state_publisher launch in rsp.launch.py

File: src/amr_description/urdf/includes/gazebo.xacro (robot description, xacro)
@@ -3,8 +3,6 @@
   <gazebo reference="base_link">
     <material>Gazebo/Red</material>
-  </gazebo>
-  <gazebo reference="base_link">
-    <plugin filename="libgz_ros2_control_system.so" name="gz_ros2_control::GazeboSystem">
-      <ros2_control_name>diff_drive</ros2_control_name>
+    <plugin filename="libgz_ros2_control-system.so" name="gz_ros2_control::GazeboSimROS2ControlPlugin">
+      <parameters>$(find amr_control)/config/controller_manager.yaml</parameters>
     </plugin>
   </gazebo>
@@ -112,27 +110,11 @@
     </sensor>
   </gazebo>
-  <gazebo reference="wheel_left_joint">
-    <collision>
-      <surface>
-        <friction>
-          <ode>
-            <mu>0.8</mu>
-            <mu2>0.8</mu2>
-          </ode>
-        </friction>
-      </surface>
-    </collision>
+  <gazebo reference="wheel_left_link">
+    <mu1>0.8</mu1>
+    <mu2>0.8</mu2>
   </gazebo>
-  <gazebo reference="wheel_right_joint">
-    <collision>
-      <surface>
-        <friction>
-          <ode>
-            <mu>0.8</mu>
-            <mu2>0.8</mu2>
-          </ode>
-        </friction>
-      </surface>
-    </collision>
+  <gazebo reference="wheel_right_link">
+    <mu1>0.8</mu1>
+    <mu2>0.8</mu2>
   </gazebo>
   <gazebo reference="caster_front_link">

File: src/amr_description/urdf/includes/transmissions.xacro (robot description, xacro)
@@ -3,5 +3,5 @@
   <ros2_control name="diff_drive" type="system">
     <hardware>
-      <plugin>gz_ros2_control/GazeboSystem</plugin>
+      <plugin>gz_ros2_control/GazeboSimSystem</plugin>
     </hardware>
     <joint name="wheel_left_joint">
@@ -16,15 +16,3 @@
     </joint>
   </ros2_control>
-  <transmission name="wheel_left_trans">
-    <type>transmission_interface/SimpleTransmission</type>
-    <joint>wheel_left_joint</joint>
-    <actuator name="wheel_left_actuator"/>
-    <mechanicalReduction>1</mechanicalReduction>
-  </transmission>
-  <transmission name="wheel_right_trans">
-    <type>transmission_interface/SimpleTransmission</type>
-    <joint>wheel_right_joint</joint>
-    <actuator name="wheel_right_actuator"/>
-    <mechanicalReduction>1</mechanicalReduction>
-  </transmission>
 </robot>
