Commit message: fix(description): honor robot_description arg, align wheel track
rsp.launch.py declared a robot_description launch argument but always
processed the hardcoded default xacro, silently ignoring the value
every caller passed. Switch to Command substitution so the selected
xacro is expanded at launch time.

Kinematics: wheel_y_offset 0.13 -> 0.15 so the URDF wheel track
(2 * 0.15 = 0.30 m) matches diff_drive_controller wheel_separation,
which the README and spec require.

File: src/amr_description/urdf/includes/properties.xacro (robot description, xacro)
@@ -5,4 +5,6 @@
        ============================================================ -->
   <xacro:property name="chassis_length" value="0.28"/>
+  <!-- Chassis half-width 0.11 m < wheel_y_offset 0.15 m:
+       wheels protrude outside the chassis, as expected -->
   <xacro:property name="chassis_width" value="0.22"/>
   <xacro:property name="chassis_height" value="0.04"/>
@@ -15,5 +17,7 @@
   <xacro:property name="wheel_length" value="0.02"/>
   <xacro:property name="wheel_mass" value="0.5"/>
-  <xacro:property name="wheel_y_offset" value="0.13"/>
+  <!-- Wheel track: 2 * wheel_y_offset = 0.30 m, must match
+       diff_drive_controller.yaml wheel_separation -->
+  <xacro:property name="wheel_y_offset" value="0.15"/>
   <xacro:property name="wheel_z_offset" value="-0.04"/>
   <xacro:property name="wheel_effort" value="100"/>
